File: Schematics/HerbBoxKicad/HerbBoxKicad.sch (KiCad schematic (older format))
At the start: 24 parts, among them J1 Capacitive Soil Moisture Sens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, J2 Capacitive Soil Moisture Sens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, J3 Capacitive Soil Moisture Sens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, K1 FINDER-32.21-x000, K2 FINDER-32.21-x000, K3 FINDER-32.21-x000, K4 FINDER-32.21-x000, M1 PUMP3, M2 PUMP2, M3 PUMP1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

Commit message: NodeMCU : Move TX line from D8 to D0
D8 needs to be low when booting but the Arduino Nano pull it high so the
NodeMCU doesn't boot properly when the TX line is connected. Using pin
D0 leaves D8 free when booting and allows everything to work properly.

Signed-off-by: Maxime Chretien (MixLeNain) <mchretien@linuxmail.org>
Connections:
- net at A1.2 (D0/RX): now also U1.30 (D0(GPIO16)); no longer U1.20 (D8(GPIO15))
Changed lines of the file:
@@
 Title "HerbBox2.0"
 Date "2021-02-01"
-Rev "v1.1"
+Rev "v1.2"
 Comp "Zoomacom / OpenFactory"
 Comment1 "mchretien@linuxmail.org"
@@
 $EndComp
 Wire Wire Line
-	4600 2550 4600 3550
-Wire Wire Line
 	4550 2650 6150 2650
 Wire Wire Line
@@
 Wire Wire Line
 	6250 950  6250 1450
-Wire Wire Line
-	4600 2550 6150 2550
-Wire Wire Line
-	2950 3550 4600 3550
 $Comp
 L Sensor_Temperature:DS18B20 U4
@@
 NoConn ~ 1350 2850
 NoConn ~ 1350 2550
-NoConn ~ 2950 2550
 NoConn ~ 2950 3050
 NoConn ~ 2950 3150
@@
 NoConn ~ 2950 3650
 NoConn ~ 2950 3750
+Wire Wire Line
+	2950 2550 6150 2550
+NoConn ~ 2950 3550
 $EndSCHEMATC
